File: theremin_project/Theremin_Project.kicad_pcb (KiCad board)
At the start: 2 copper layers, 19 parts, among them U1 MCP602, U4 Opamp_Dual, U5 ESP32-WROOM-32

Commit message: layout and sch
Parts:
- removed U5: ESP32-WROOM-32, RF_Module:ESP32-WROOM-32
- added AE1: Antenna, RF_Antenna:Texas_SWRA416_868MHz_915MHz, F.Cu at (71.9, 85.2)
- added C5: 1uF, Capacitor_SMD:C_0201_0603Metric, F.Cu at (109.2, 102.2)
- added C6: 1uF, Capacitor_SMD:C_0201_0603Metric, F.Cu at (112.1, 97.2)
- added J1: Conn_01x02_Pin, Connector_PinHeader_2.54mm:PinHeader_1x02_P2.54mm_Vertical, F.Cu at (116.8, 88.9)
- added J2: TYPE-C-31-M-12, TYPE-C-31-M-12:HRO_TYPE-C-31-M-12, F.Cu at (152.4, 104.1)
- added J3: Conn_01x01_Pin, Connector_PinHeader_1.00mm:PinHeader_1x01_P1.00mm_Vertical, F.Cu at (101.6, 99.1)
- added R11: RM2012A-502_104-PBVW10, RM2012A-502_104-PBVW10:RESCAXE_RM2012-4N, F.Cu at (146.8, 115.6)
- added R9: 100k, Resistor_THT:R_Axial_DIN0204_L3.6mm_D1.6mm_P1.90mm_Vertical, F.Cu at (119.4, 101.6)
- added U8: NCP164CSN330T1G, NCP:FP-NCP164CSN330T1G_OSI, F.Cu at (113.0, 100.6)
- U1: value MCP602 -> AD8001AR; footprint Package_CSP:LFCSP-8_2x2mm_P0.5mm -> Package_SO:SOIC-8_3.9x4.9mm_P1.27mm
- U2: value ~ -> HEF4093B; footprint Button_Switch_SMD:SW_DIP_SPSTx07_Slide_6.7x19.34mm_W6.73mm_P2.54mm_LowProfile_JPin -> HEF4093BP_652:DIP254P762X420-14
- U3: value ~ -> AD8001AR; footprint Button_Switch_SMD:SW_DIP_SPSTx07_Slide_6.7x19.34mm_W6.73mm_P2.54mm_LowProfile_JPin -> Package_SO:SOIC-8_3.9x4.9mm_P1.27mm
- U4: value Opamp_Dual -> ESP32-S2-SOLO-N4R2; footprint Package_DIP:DIP-8-16_W7.62mm -> esp32:MOD41_ESP32-S2-SOLO_EXP
- moved U4 86.0 mm to (134.0, 96.5), turned to 0 degrees
- moved C3 79.7 mm to (144.6, 121.9), turned to 180 degrees
- moved C4 74.3 mm to (139.5, 124.5), turned to -90 degrees
- moved C1 69.2 mm to (101.6, 104.1), turned to 180 degrees
- moved R6 68.9 mm to (137.3, 121.9)
- moved R7 66.1 mm to (124.5, 113.7), turned to 180 degrees
- moved R5 63.1 mm to (120.1, 118.7)
- moved R1 62.4 mm to (101.6, 109.2)
- moved U1 60.0 mm to (129.6, 118.7)
- moved RV1 59.8 mm to (99.1, 117.9)
- moved R8 59.4 mm to (124.5, 126.4), turned to 180 degrees
- moved R10 57.0 mm to (142.4, 124.5), turned to -90 degrees
- moved R2 56.9 mm to (101.6, 106.7)
- moved R4 56.3 mm to (122.0, 121.3), turned to 180 degrees
- moved C2 50.7 mm to (99.4, 127.0), turned to 180 degrees
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Connections:
- C1 pad 1: Net-(AE1-A) -> Net-(J3-Pin_1)
- C3 pad 1: Net-(C3-Pad1) -> Net-(U3-+)
- R2 pad 2: Net-(AE1-A) -> Net-(J3-Pin_1)
- R4 pad 2: Net-(U3-K=CD) -> Net-(R4-Pad2)
- RV1 pad 2: Net-(U3-K=CD) -> Net-(R4-Pad2)
- RV1 pad 3: Net-(U3-K=CD) -> Net-(R4-Pad2)
- U1 pad 1: Net-(R6-Pad1) -> unconnected-(U1-NC-Pad1)
- U1 pad 4: (no net) -> GND
- U1 pad 5: (no net) -> unconnected-(U1-NC-Pad5)
- U1 pad 6: (no net) -> Net-(R6-Pad1)
- U1 pad 7: (no net) -> +5V
- U1 pad 8: (no net) -> unconnected-(U1-NC-Pad8)
- U2 pad 1: unconnected-(U2-A-Pad1) -> Net-(U2-Pad1)
- U2 pad 10: unconnected-(U2-L=EF-Pad10) -> (no net)
- U2 pad 11: unconnected-(U2-M=GH-Pad11) -> (no net)
- U2 pad 12: unconnected-(U2-G-Pad12) -> (no net)
- U2 pad 13: unconnected-(U2-M-Pad13) -> (no net)
- U2 pad 14: unconnected-(U2-Vdd-Pad14) -> +5V
- U2 pad 2: unconnected-(U2-B-Pad2) -> Net-(J3-Pin_1)
- U2 pad 3: unconnected-(U2-J=AB-Pad3) -> Net-(R1-Pad1)
- U2 pad 4: unconnected-(U2-K=CD-Pad4) -> Net-(R4-Pad2)
- U2 pad 5: unconnected-(U2-C-Pad5) -> Net-(U2-Pad5)
- U2 pad 6: unconnected-(U2-D-Pad6) -> Net-(C2-Pad1)
- U2 pad 7: unconnected-(U2-Vss-Pad7) -> GND
- U2 pad 8: unconnected-(U2-E-Pad8) -> (no net)
- U2 pad 9: unconnected-(U2-F-Pad9) -> (no net)
- U3 pad 2: unconnected-(U3-B-Pad2) -> Net-(U3--)
- U3 pad 3: unconnected-(U3-J=AB-Pad3) -> Net-(U3-+)
- U3 pad 4: Net-(U3-K=CD) -> GND
- U3 pad 6: unconnected-(U3-D-Pad6) -> Net-(U3--)
- U3 pad 7: unconnected-(U3-Vss-Pad7) -> +5V
- U4 pad 1: (no net) -> GND
- U4 pad 2: (no net) -> Net-(U4-3V3)
- U4 pad 3: (no net) -> unconnected-(U4-EN-Pad3)
- U4 pad 4: GND -> unconnected-(U4-IO4-Pad4)
- U4 pad 5: (no net) -> Net-(U3--)
- U4 pad 6: (no net) -> unconnected-(U4-IO6-Pad6)
- U4 pad 7: (no net) -> unconnected-(U4-IO7-Pad7)
- U4 pad 8: +5V -> unconnected-(U4-IO15-Pad8)
Routing:
- net GND: track 31.5 -> 200.5 mm, vias 0 -> 2
- net +5V: track 0.00 -> 61.0 mm
- net Net-(U3--): track 0.00 -> 34.4 mm
- net Net-(R4-Pad2): track 0.00 -> 30.2 mm
- net Net-(J2-DN2): track 0.00 -> 28.3 mm, vias 0 -> 2
- net Net-(J2-DP2): track 0.00 -> 25.7 mm, vias 0 -> 2
- net Net-(U4-3V3): track 0.00 -> 18.6 mm
- net Net-(J3-Pin_1): track 0.00 -> 16.2 mm
- net Net-(U3-K=CD): track 15.8 -> 0.00 mm, vias 2 -> 0
- net Net-(U3-+): track 0.00 -> 14.9 mm
- net Net-(R1-Pad2): track 18.2 -> 3.33 mm
- net Net-(R3-Pad1): track 22.1 -> 7.26 mm, vias 1 -> 0
- net Net-(R1-Pad1): track 8.56 -> 23.1 mm
- net Net-(AE1-A): track 13.4 -> 0.00 mm, vias 2 -> 0
- net Net-(U1--): track 7.16 -> 16.1 mm, vias 2 -> 0
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- added copper zone on B.Cu, net GND
Other:
- board outline added: 63.5 x 48.3 mm
